Commit message: Add models for Zivid 3 XL250

File: zivid_description/urdf/macros/zivid_camera.xacro (robot description, xacro)
@@ -5,4 +5,6 @@
     <xacro:macro name="zivid_camera" params="prefix model field_of_view">
         <xacro:property name="fov_filename" value="" />
+        <xacro:property name="visual_mesh" value="zivid_2_plus.stl" />
+        <xacro:property name="collision_mesh" value="zivid_2_plus_convex_hull.stl" />
         <xacro:if value="${model == 'ZIVID_2_M70'}">
             <xacro:property name="optical_center" value="0.04802 0.03084 0.0295" />
@@ -45,4 +47,11 @@
             <xacro:property name="fov_filename" value="zivid_2_plus_m130_fov" />
         </xacro:if>
+        <xacro:if value="${model == 'ZIVID_3_XL250'}">
+            <xacro:property name="optical_center" value="0.047 0.10050 0.0365" />
+            <xacro:property name="optical_angle_deg" value="0.0" />
+            <xacro:property name="fov_filename" value="zivid_3_xl250_fov" />
+            <xacro:property name="visual_mesh" value="zivid_3.stl" />
+            <xacro:property name="collision_mesh" value="zivid_3_convex_hull.stl" />
+        </xacro:if>
         <!-- Make xacro error out if the provided camera model was not recognized -->
         <xacro:if value="${fov_filename == ''}">
@@ -55,5 +64,5 @@
                 <origin xyz="0 0 0" rpy="0 0 ${0.5*pi}"/>
                 <geometry>
-                    <mesh filename="package://zivid_description/meshes/visual/zivid_2_plus.stl"/>
+                    <mesh filename="package://zivid_description/meshes/visual/${visual_mesh}"/>
                 </geometry>
                 <material name="zivid_gray"/>
@@ -63,5 +72,5 @@
                 <origin xyz="0 0 0" rpy="0 0 ${0.5*pi}"/>
                 <geometry>
-                    <mesh filename="package://zivid_description/meshes/collision/zivid_2_plus_convex_hull.stl"/>
+                    <mesh filename="package://zivid_description/meshes/collision/${collision_mesh}"/>
                 </geometry>
             </collision>
