Commit message: Rename files to indicate camera type
As the Zivid Two launched, it is needed to differntiate between the
types.

File: zivid_description/urdf/macros/zivid_one_plus_camera.xacro (robot description, xacro)
@@ -5,5 +5,5 @@
         <color rgba="0.25 0.25 0.25 1"/>
     </material>
-    <xacro:macro name="zivid_camera" params="prefix">
+    <xacro:macro name="zivid_one_plus_camera" params="prefix">
         <!-- Zivid Base Link -->
         <link name="${prefix}base_link">

Commit message: Remove projector frame
Requested by Zivid as it might cause confusion

File: zivid_description/urdf/macros/zivid_one_plus_camera.xacro (robot description, xacro)
@@ -26,5 +26,4 @@
         <!-- Zivid Optical (Measurement) and Projector Frames -->
         <link name="${prefix}optical_frame"/>
-        <link name="${prefix}projector_frame"/>
         <!-- Zivid Optical (Measurement) and Projector Joints -->
         <joint name="${prefix}optical_joint" type="fixed">
@@ -33,9 +32,4 @@
             <child link="${prefix}optical_frame"/>
         </joint>
-        <joint name="${prefix}projector_joint" type="fixed">
-            <origin xyz="-0.0030 -0.0758 0.0445" rpy="-${0.5*pi} 0 -${0.5*pi}"/>
-            <parent link="${prefix}base_link"/>
-            <child link="${prefix}projector_frame"/>
-        </joint>
     </xacro:macro>
 </robot>

Commit message: Update macro and launch files
The macro now supports the S, M, and L types of the ZIvid One+. Launch
files to load, and/or view the different variants have been included.

File: zivid_description/urdf/macros/zivid_one_plus_camera.xacro (robot description, xacro)
@@ -1,9 +1,17 @@
 <?xml version="1.0"?>
 <robot xmlns:xacro="http://ros.org/wiki/xacro">
-    <!-- Properties -->
+    <!-- Zivid One+ Types: Can be accessed globally and used as identifiers -->
+    <xacro:property name="Zivid_One_Plus_S" value="0" scope="global" />
+    <xacro:property name="Zivid_One_Plus_M" value="1" scope="global" />
+    <xacro:property name="Zivid_One_Plus_L" value="2" scope="global" />
+    <!-- Zivid One+ Optical Frame Angles -->
+    <xacro:property name="angle_type_s" value="15.0" />
+    <xacro:property name="angle_type_m" value="8.5" />
+    <xacro:property name="angle_type_l" value="6.0" />
+    <!-- Material Properties -->
     <material name="zivid_gray">
         <color rgba="0.25 0.25 0.25 1"/>
     </material>
-    <xacro:macro name="zivid_one_plus_camera" params="prefix">
+    <xacro:macro name="zivid_one_plus_camera" params="prefix type">
         <!-- Zivid Base Link -->
         <link name="${prefix}base_link">
@@ -24,9 +32,19 @@
             </collision>
         </link>
-        <!-- Zivid Optical (Measurement) and Projector Frames -->
+        <!-- Zivid Optical Frame (Measurement Frame)-->
         <link name="${prefix}optical_frame"/>
-        <!-- Zivid Optical (Measurement) and Projector Joints -->
+        <!-- Set the angle of the optical frame based on the type -->
+        <xacro:if value="${type == Zivid_One_Plus_S}" >
+            <xacro:property name="optical_frame_angle" value="${angle_type_s}" />
+        </xacro:if>
+        <xacro:if value="${type == Zivid_One_Plus_M}" >
+            <xacro:property name="optical_frame_angle" value="${angle_type_m}" />
+        </xacro:if>
+        <xacro:if value="${type == Zivid_One_Plus_L}" >
+            <xacro:property name="optical_frame_angle" value="${angle_type_l}" />
+        </xacro:if>
+        <!-- Zivid Optical (Measurement) Joint -->
         <joint name="${prefix}optical_joint" type="fixed">
-            <origin xyz="0.065 0.062 0.0445" rpy="-${0.5*pi} 0 -${0.5*pi + 8.5/180*pi}"/>
+            <origin xyz="0.065 0.062 0.0445" rpy="-${0.5*pi} 0 -${0.5*pi + optical_frame_angle/180*pi}"/>
             <parent link="${prefix}base_link"/>
             <child link="${prefix}optical_frame"/>

File: zivid_description/urdf/zivid_one_plus_l_camera.urdf.xacro (robot description, xacro)
@@ -2,4 +2,4 @@
 <robot name="zivid_one_plus_camera_robot" xmlns:xacro="http://www.ros.org/wiki/xacro">
     <xacro:include filename="$(find zivid_description)/urdf/macros/zivid_one_plus_camera.xacro"/>
-    <xacro:zivid_one_plus_camera prefix=""/>
+    <xacro:zivid_one_plus_camera prefix="" type="${Zivid_One_Plus_L}"/>
 </robot>

Commit message: Reduce amount of xacro and launch files
 Instead the launch files and xacro's accept a type argument

File: zivid_description/urdf/macros/zivid_one_plus_camera.xacro (robot description, xacro)
@@ -1,16 +1,8 @@
 <?xml version="1.0"?>
 <robot xmlns:xacro="http://ros.org/wiki/xacro">
-    <!-- Zivid One+ Types: Can be accessed globally and used as identifiers -->
-    <xacro:property name="Zivid_One_Plus_S" value="0" scope="global" />
-    <xacro:property name="Zivid_One_Plus_M" value="1" scope="global" />
-    <xacro:property name="Zivid_One_Plus_L" value="2" scope="global" />
     <!-- Zivid One+ Optical Frame Angles -->
     <xacro:property name="angle_type_s" value="15.0" />
     <xacro:property name="angle_type_m" value="8.5" />
     <xacro:property name="angle_type_l" value="6.0" />
-    <!-- Material Properties -->
-    <material name="zivid_gray">
-        <color rgba="0.25 0.25 0.25 1"/>
-    </material>
     <xacro:macro name="zivid_one_plus_camera" params="prefix type">
         <!-- Zivid Base Link -->
@@ -35,11 +27,11 @@
         <link name="${prefix}optical_frame"/>
         <!-- Set the angle of the optical frame based on the type -->
-        <xacro:if value="${type == Zivid_One_Plus_S}" >
+        <xacro:if value="${type == 'ZIVID_ONE_PLUS_S'}" >
             <xacro:property name="optical_frame_angle" value="${angle_type_s}" />
         </xacro:if>
-        <xacro:if value="${type == Zivid_One_Plus_M}" >
+        <xacro:if value="${type == 'ZIVID_ONE_PLUS_M'}" >
             <xacro:property name="optical_frame_angle" value="${angle_type_m}" />
         </xacro:if>
-        <xacro:if value="${type == Zivid_One_Plus_L}" >
+        <xacro:if value="${type == 'ZIVID_ONE_PLUS_L'}" >
             <xacro:property name="optical_frame_angle" value="${angle_type_l}" />
         </xacro:if>
