Commit message: Add URDF/Xacro for Zivid cameras
Add a new package `zivid_description` containing URDF/Xacro files for
Zivid cameras.

Add new launch files to the sample package to launch a Zivid camera with
the URDF. Modify existing launch files to also load the URDF.
Additionally, change the Zivid RViz configuration to use the robot
description.

This way, when launching the Zivid camera with RViz, the camera will
appear in the scene. Point clouds published from captures will be shown
in the RViz scene appropriately placed in relation to the camera.

This commit builds on top of pull request #17. The following changes are
made here compared to pull request #17:

- Convert to ROS2.
- Add new visual and collision mesh for Zivid 2/2+/2+R cameras.
- Add FOV frustum meshes for the different camera models (toggleable).
- Add physical parameters for the Zivid camera models, for appropriate
  placement of the point cloud in relation to the camera.
- Remove Zivid One+ support.
- Make Xacro error out with a reasonable error message when specifying
  an unknown model.
- Rename argument type -> model.
- Move launch files to `zivid_samples`.

File: zivid_description/urdf/zivid_materials.xacro (robot description, xacro)
@@ -1,7 +1,9 @@
 <?xml version="1.0"?>
 <robot>
-    <!-- Material Properties -->
     <material name="zivid_gray">
         <color rgba="0.25 0.25 0.25 1"/>
     </material>
+    <material name="zivid_fov">
+        <color rgba="0.15 0.6 1.0 0.5"/>
+    </material>
 </robot>

Commit message: Update URDF and convert to ROS2
- Add new visual and collision mesh for Zivid 2 cameras.
- Add parameters for individual Zivid camera models.
- Add FOV frustum meshes for different models (toggleable).
- Remove Zivid One+ support.
- Rename argument type -> model.
- Make xacro error out with a reasonable error message when specifying an unknown model.

File: zivid_description/urdf/zivid_materials.xacro (robot description, xacro)
@@ -5,3 +5,6 @@
         <color rgba="0.25 0.25 0.25 1"/>
     </material>
+    <material name="zivid_fov">
+        <color rgba="0.15 0.6 1.0 0.5"/>
+    </material>
 </robot>
